File: Station/Hardware/Station-Hardware-ver-01/Station-Hardware-ver-01.kicad_sch (KiCad schematic)
At the start: 28 parts, among them J1 Barrel_Jack, J2 Conn_01x03_Male, J3 Conn_01x03_Male, J4 4P4C, J5 4P4C, J6 Conn_01x03_Male, U1 YAAJ_BluePill, U2 DS3231_Full_Pinout, U3 SX1278_Minimal, U4 MCP6002-xP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

Commit message: pcb design for the station
Parts:
- C1, C6: value (none) -> 68n; footprint (none) -> Capacitor_SMD:C_0805_2012Metric_Pad1.18x1.45mm_HandSolder
- C2: value (none) -> 10n; footprint (none) -> Capacitor_SMD:C_0805_2012Metric_Pad1.18x1.45mm_HandSolder
- C3: value (none) -> 4.7n; footprint (none) -> Capacitor_SMD:C_0805_2012Metric_Pad1.18x1.45mm_HandSolder
- C4: value (none) -> 3.3n; footprint (none) -> Capacitor_SMD:C_0805_2012Metric_Pad1.18x1.45mm_HandSolder
- C5: value (none) -> 2.2n; footprint (none) -> Capacitor_SMD:C_0805_2012Metric_Pad1.18x1.45mm_HandSolder
- C7: value (none) -> 0.1u; footprint (none) -> Capacitor_SMD:CP_Elec_4x5.4
- C8: value (none) -> 1u; footprint (none) -> Capacitor_SMD:CP_Elec_4x5.4
- R1: value (none) -> 3k; footprint (none) -> Resistor_SMD:R_1206_3216Metric_Pad1.30x1.75mm_HandSolder
- R2, R5: value (none) -> 33k; footprint (none) -> Resistor_SMD:R_1206_3216Metric_Pad1.30x1.75mm_HandSolder
- R3: value (none) -> 680; footprint (none) -> Resistor_SMD:R_1206_3216Metric_Pad1.30x1.75mm_HandSolder
- R4: value (none) -> 3.3k; footprint (none) -> Resistor_SMD:R_1206_3216Metric_Pad1.30x1.75mm_HandSolder
- R6: value (none) -> 4.7k; footprint (none) -> Resistor_SMD:R_1206_3216Metric_Pad1.30x1.75mm_HandSolder
- R7: value (none) -> 240; footprint (none) -> Resistor_SMD:R_1206_3216Metric_Pad1.30x1.75mm_HandSolder
- R8: value (none) -> 390; footprint (none) -> Resistor_SMD:R_1206_3216Metric_Pad1.30x1.75mm_HandSolder
- U1: value YAAJ_BluePill -> (none); footprint KiCAD_STM32_BluePill:YAAJ_BluePill_1 -> (none)
Changed lines of the file:
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@@
       (effects (font (size 1.27 1.27)) (justify left))
     )
-    (property "Value" "" (id 1) (at 124.206 138.4299 0)
-      (effects (font (size 1.27 1.27)) (justify left))
-    )
-    (property "Footprint" "" (id 2) (at 120.142 137.16 90)
+    (property "Value" "33k" (id 1) (at 124.206 138.4299 0)
+      (effects (font (size 1.27 1.27)) (justify left))
+    )
+    (property "Footprint" "Resistor_SMD:R_1206_3216Metric_Pad1.30x1.75mm_HandSolder" (id 2) (at 120.142 137.16 90)
       (effects (font (size 1.27 1.27)) hide)
     )
@@
     (in_bom yes) (on_board yes)
     (property "Reference" "C1" (id 0) (at 127 101.6 90))
-    (property "Value" "" (id 1) (at 127 103.505 90))
-    (property "Footprint" "" (id 2) (at 130.81 96.8248 0)
+    (property "Value" "68n" (id 1) (at 127 103.505 90))
+    (property "Footprint" "Capacitor_SMD:C_0805_2012Metric_Pad1.18x1.45mm_HandSolder" (id 2) (at 130.81 96.8248 0)
       (effects (font (size 1.27 1.27)) hide)
     )
@@
       (effects (font (size 1.27 1.27)) (justify left))
     )
-    (property "Value" "" (id 1) (at 53.34 114.3 0)
-      (effects (font (size 1.27 1.27)) (justify left))
-    )
-    (property "Footprint" "" (id 2) (at 59.69 113.03 0)
+    (property "Value" "0.1u" (id 1) (at 53.34 114.3 0)
+      (effects (font (size 1.27 1.27)) (justify left))
+    )
+    (property "Footprint" "Capacitor_SMD:CP_Elec_4x5.4" (id 2) (at 59.69 113.03 0)
       (effects (font (size 1.27 1.27)) hide)
     )
@@
       (effects (font (size 1.27 1.27)) (justify left))
     )
-    (property "Value" "" (id 1) (at 90.17 114.3 0)
-      (effects (font (size 1.27 1.27)) (justify left))
-    )
-    (property "Footprint" "" (id 2) (at 87.63 113.03 0)
+    (property "Value" "1u" (id 1) (at 90.17 114.3 0)
+      (effects (font (size 1.27 1.27)) (justify left))
+    )
+    (property "Footprint" "Capacitor_SMD:CP_Elec_4x5.4" (id 2) (at 87.63 113.03 0)
       (effects (font (size 1.27 1.27)) hide)
     )
@@
       (effects (font (size 1.27 1.27)) (justify left))
     )
-    (property "Value" "" (id 1) (at 198.12 87.6299 0)
-      (effects (font (size 1.27 1.27)) (justify left))
-    )
-    (property "Footprint" "" (id 2) (at 195.2752 90.17 0)
+    (property "Value" "10n" (id 1) (at 198.12 87.6299 0)
+      (effects (font (size 1.27 1.27)) (justify left))
+    )
+    (property "Footprint" "Capacitor_SMD:C_0805_2012Metric_Pad1.18x1.45mm_HandSolder" (id 2) (at 195.2752 90.17 0)
       (effects (font (size 1.27 1.27)) hide)
     )
@@
     (in_bom yes) (on_board yes)
     (property "Reference" "R7" (id 0) (at 82.55 107.95 0))
-    (property "Value" "" (id 1) (at 82.55 110.49 0))
-    (property "Footprint" "" (id 2) (at 80.518 109.22 90)
+    (property "Value" "240" (id 1) (at 82.55 110.49 0))
+    (property "Footprint" "Resistor_SMD:R_1206_3216Metric_Pad1.30x1.75mm_HandSolder" (id 2) (at 80.518 109.22 90)
       (effects (font (size 1.27 1.27)) hide)
     )
@@
       (effects (font (size 1.27 1.27)) (justify left))
     )
-    (property "Value" "" (id 1) (at 209.55 87.6299 0)
-      (effects (font (size 1.27 1.27)) (justify left))
-    )
-    (property "Footprint" "" (id 2) (at 206.7052 90.17 0)
+    (property "Value" "4.7n" (id 1) (at 209.55 87.6299 0)
+      (effects (font (size 1.27 1.27)) (justify left))
+    )
+    (property "Footprint" "Capacitor_SMD:C_0805_2012Metric_Pad1.18x1.45mm_HandSolder" (id 2) (at 206.7052 90.17 0)
       (effects (font (size 1.27 1.27)) hide)
     )
@@
     (in_bom yes) (on_board yes)
     (property "Reference" "R6" (id 0) (at 200.025 140.97 90))
-    (property "Value" "" (id 1) (at 200.025 143.51 90))
-    (property "Footprint" "" (id 2) (at 200.025 140.208 90)
+    (property "Value" "4.7k" (id 1) (at 200.025 143.51 90))
+    (property "Footprint" "Resistor_SMD:R_1206_3216Metric_Pad1.30x1.75mm_HandSolder" (id 2) (at 200.025 140.208 90)
       (effects (font (size 1.27 1.27)) hide)
     )
@@
     (in_bom yes) (on_board yes)
     (property "Reference" "R8" (id 0) (at 82.55 115.57 0))
-    (property "Value" "" (id 1) (at 82.55 118.11 0))
-    (property "Footprint" "" (id 2) (at 76.962 116.84 90)
+    (property "Value" "390" (id 1) (at 82.55 118.11 0))
+    (property "Footprint" "Resistor_SMD:R_1206_3216Metric_Pad1.30x1.75mm_HandSolder" (id 2) (at 76.962 116.84 90)
       (effects (font (size 1.27 1.27)) hide)
     )
@@
     (in_bom yes) (on_board yes)
     (property "Reference" "R4" (id 0) (at 241.3 95.25 90))
-    (property "Value" "" (id 1) (at 241.3 97.155 90))
-    (property "Footprint" "" (id 2) (at 241.3 94.488 90)
+    (property "Value" "3.3k" (id 1) (at 241.3 97.155 90))
+    (property "Footprint" "Resistor_SMD:R_1206_3216Metric_Pad1.30x1.75mm_HandSolder" (id 2) (at 241.3 94.488 90)
       (effects (font (size 1.27 1.27)) hide)
     )
@@
       (effects (font (size 1.27 1.27)) (justify left))
     )
-    (property "Value" "YAAJ_BluePill" (id 1) (at 55.3594 91.44 0)
-      (effects (font (size 1.27 1.27)) (justify left))
-    )
-    (property "Footprint" "KiCAD_STM32_BluePill:YAAJ_BluePill_1" (id 2) (at 51.435 30.48 90)
+    (property "Value" "" (id 1) (at 55.3594 91.44 0)
+      (effects (font (size 1.27 1.27)) (justify left))
+    )
+    (property "Footprint" "" (id 2) (at 51.435 30.48 90)
       (effects (font (size 1.27 1.27)) hide)
     )
@@
       (effects (font (size 1.27 1.27)) (justify left))
     )
-    (property "Value" "" (id 1) (at 232.41 87.6299 0)
-      (effects (font (size 1.27 1.27)) (justify left))
-    )
-    (property "Footprint" "" (id 2) (at 229.5652 90.17 0)
+    (property "Value" "2.2n" (id 1) (at 232.41 87.6299 0)
+      (effects (font (size 1.27 1.27)) (justify left))
+    )
+    (property "Footprint" "Capacitor_SMD:C_0805_2012Metric_Pad1.18x1.45mm_HandSolder" (id 2) (at 229.5652 90.17 0)
       (effects (font (size 1.27 1.27)) hide)
     )
@@
       (effects (font (size 1.27 1.27)) (justify left))
     )
-    (property "Value" "" (id 1) (at 124.206 85.0899 0)
-      (effects (font (size 1.27 1.27)) (justify left))
-    )
-    (property "Footprint" "" (id 2) (at 120.142 83.82 90)
+    (property "Value" "3k" (id 1) (at 124.206 85.0899 0)
+      (effects (font (size 1.27 1.27)) (justify left))
+    )
+    (property "Footprint" "Resistor_SMD:R_1206_3216Metric_Pad1.30x1.75mm_HandSolder" (id 2) (at 120.142 83.82 90)
       (effects (font (size 1.27 1.27)) hide)
     )
@@
     (in_bom yes) (on_board yes)
     (property "Reference" "C6" (id 0) (at 128.27 152.4 90))
-    (property "Value" "" (id 1) (at 128.27 154.305 90))
-    (property "Footprint" "" (id 2) (at 132.08 147.6248 0)
+    (property "Value" "68n" (id 1) (at 128.27 154.305 90))
+    (property "Footprint" "Capacitor_SMD:C_0805_2012Metric_Pad1.18x1.45mm_HandSolder" (id 2) (at 132.08 147.6248 0)
       (effects (font (size 1.27 1.27)) hide)
     )
@@
       (effects (font (size 1.27 1.27)) (justify left))
     )
-    (property "Value" "" (id 1) (at 133.731 85.0899 0)
-      (effects (font (size 1.27 1.27)) (justify left))
-    )
-    (property "Footprint" "" (id 2) (at 129.667 83.82 90)
+    (property "Value" "33k" (id 1) (at 133.731 85.0899 0)
+      (effects (font (size 1.27 1.27)) (justify left))
+    )
+    (property "Footprint" "Resistor_SMD:R_1206_3216Metric_Pad1.30x1.75mm_HandSolder" (id 2) (at 129.667 83.82 90)
       (effects (font (size 1.27 1.27)) hide)
     )
@@
       (effects (font (size 1.27 1.27)) (justify left))
     )
-    (property "Value" "" (id 1) (at 220.98 87.6299 0)
-      (effects (font (size 1.27 1.27)) (justify left))
-    )
-    (property "Footprint" "" (id 2) (at 218.1352 90.17 0)
+    (property "Value" "3.3n" (id 1) (at 220.98 87.6299 0)
+      (effects (font (size 1.27 1.27)) (justify left))
+    )
+    (property "Footprint" "Capacitor_SMD:C_0805_2012Metric_Pad1.18x1.45mm_HandSolder" (id 2) (at 218.1352 90.17 0)
       (effects (font (size 1.27 1.27)) hide)
     )
@@
     (in_bom yes) (on_board yes)
     (property "Reference" "R3" (id 0) (at 187.96 75.565 90))
-    (property "Value" "" (id 1) (at 187.96 77.47 90))
-    (property "Footprint" "" (id 2) (at 187.96 81.788 90)
+    (property "Value" "680" (id 1) (at 187.96 77.47 90))
+    (property "Footprint" "Resistor_SMD:R_1206_3216Metric_Pad1.30x1.75mm_HandSolder" (id 2) (at 187.96 81.788 90)
       (effects (font (size 1.27 1.27)) hide)
     )
@@
     )
     (path "/a3f9c6b6-1661-4aed-910d-16d5cf883aed"
-      (reference "U1") (unit 1) (value "YAAJ_BluePill") (footprint "KiCAD_STM32_BluePill:YAAJ_BluePill_1")
+      (reference "U1") (unit 1) (value "YAAJ_BluePill") (footprint "KiCAD-STM32BluePill:YAAJ_BluePill_1")
     )
     (path "/cfd91841-080f-43ed-a17b-46bda37a2e87"
@@
     )
     (path "/77006be8-e871-4875-98bd-df9b9f9c71da"
-      (reference "U6") (unit 1) (value "LM317_TO-220") (footprint "Package_TO_SOT_THT:TO-220-3_Horizontal_TabDown")
-    )
-  )
+      (reference "U6") (unit 1) (value "LM317_TO-220") (footprint "Package_TO_SOT_THT:TO-220-3_Vertical")
+    )
+  )
